Commit message: Created thruster vector control, updated xacro files

File: ucf_sub/src/sub_definition/robots/ucf_robosub.urdf.xacro (robot description, xacro)
@@ -6,13 +6,15 @@
     <xacro:include filename="$(find ucf_sub_definition)/urdf/vision_cam.urdf.xacro"/>
     <sub_body />
-    <sub_thruster identifier="topStrafe" parent="base_link" xPos="0.0" yPos="0.0" zPos="-0.1542" roll="3.141" pitch="0.0" yaw="1.571"/>
-    <sub_thruster identifier="bottomStrafe" parent="base_link" xPos="0.0" yPos="0.0" zPos="0.1542" roll="0.0" pitch="0.0" yaw="-1.571"/>
-    <sub_thruster identifier="leftSurge" parent="base_link" xPos="0.0" yPos="-0.1542" zPos="0.0" roll="1.571" pitch="3.141" yaw="0.0"/>
-    <sub_thruster identifier="rightSurge" parent="base_link" xPos="0.0" yPos="0.1542" zPos="0.0" roll="-1.571" pitch="3.141" yaw="0.0"/>
-    <sub_thruster identifier="frontVertical" parent="base_link" xPos="0.1968" yPos="0" zPos="0.0" roll="0.0" pitch="-1.571" yaw="0.0"/>
-    <sub_thruster identifier="rearVertical" parent="base_link" xPos="-0.1968" yPos="0" zPos="0.0" roll="0.0" pitch="-1.571" yaw="0.0"/>
-    <sub_arm identifier="right" parent="base_link" xPos="0.359" yPos="0.0878" zPos="0.0509" roll="0.0" pitch="0.0" yaw="0.0"/>
-    <sub_arm identifier="left" parent="base_link" xPos="0.359" yPos="-0.0369" zPos="0.0509" roll="0.0" pitch="0.0" yaw="0.0"/>
-    <sub_vision_cam identifier="left" parent="base_link" xPos="0.43" yPos="-0.03" zPos="0.0" roll="0.0" pitch="0.0" yaw="0.0"/>
-    <sub_vision_cam identifier="right" parent="base_link" xPos="0.43" yPos="0.03" zPos="0.0" roll="0.0" pitch="0.0" yaw="0.0"/>
+    <sub_thruster identifier="vertical1" parent="base_link" xPos="0.11" yPos="-0.18" zPos="0.0" roll="1.571" pitch="1.571" yaw="0.0"/>
+    <sub_thruster identifier="vertical2" parent="base_link" xPos="-0.08" yPos="-0.18" zPos="0.0" roll="1.571" pitch="1.571" yaw="0.0"/>
+    <sub_thruster identifier="vertical3" parent="base_link" xPos="-0.08" yPos="0.18" zPos="0.0" roll="-1.571" pitch="1.571" yaw="0.0"/>
+    <sub_thruster identifier="vertical4" parent="base_link" xPos="0.11" yPos="0.18" zPos="0.0" roll="-1.571" pitch="1.571" yaw="0.0"/>
+    <sub_thruster identifier="horizontal1" parent="base_link" xPos="0.24" yPos="-0.19" zPos="0.0" roll="-1.571" pitch="0.0" yaw="3.927"/>
+    <sub_thruster identifier="horizontal2" parent="base_link" xPos="-0.21" yPos="-0.19" zPos="0.0" roll="1.571" pitch="0.0" yaw="-0.785"/>
+    <sub_thruster identifier="horizontal3" parent="base_link" xPos="-0.21" yPos="0.19" zPos="0.0" roll="-1.571" pitch="0.0" yaw="0.785"/>
+    <sub_thruster identifier="horizontal4" parent="base_link" xPos="0.24" yPos="0.19" zPos="0.0" roll="1.571" pitch="0.0" yaw="-3.927"/>
+    <sub_arm identifier="right" parent="base_link" xPos="0.275" yPos="0.099" zPos="-0.0623" roll="0.0" pitch="0.0" yaw="0.0"/>
+    <sub_arm identifier="left" parent="base_link" xPos="0.275" yPos="-0.0482" zPos="-0.0623" roll="0.0" pitch="0.0" yaw="0.0"/>
+    <sub_vision_cam identifier="left" parent="base_link" xPos="0.301" yPos="-0.051" zPos="0.0" roll="0.0" pitch="0.0" yaw="0.0"/>
+    <sub_vision_cam identifier="right" parent="base_link" xPos="0.301" yPos="0.051" zPos="0.0" roll="0.0" pitch="0.0" yaw="0.0"/>
 </robot>

File: ucf_sub/src/sub_definition/urdf/sub_arm.urdf.xacro (robot description, xacro)
@@ -7,5 +7,5 @@
                     <box size="0.0381 0.0509 0.05"/>
                 </geometry>
-                <origin rpy="0 0 0" xyz="0.0191 -0.0255 0.025"/>
+                <origin rpy="0 0 0" xyz="-0.01905 -0.0254 -0.03"/>
             </visual>
         </link>
@@ -26,7 +26,7 @@
 		    <parent link="${identifier}_arm_base"/>
 		    <child link="${identifier}_arm_main"/>
-		    <origin xyz="0.019 -0.0254 0.0631" rpy="0 0 0"/>
+		    <origin xyz="-0.0191 -0.0254 -0.076" rpy="0 0 0"/>
 		    <axis xyz="0 1 0"/>
-		    <limit lower="-1.57" upper="0.2" effort="2.8" velocity="20"/>
+		    <limit effort="2.8" lower="-1.57" upper="0.2" velocity="20"/>
 		</joint>
     </xacro:macro>

File: ucf_sub/src/sub_definition/urdf/sub_body.urdf.xacro (robot description, xacro)
@@ -5,5 +5,5 @@
             <visual>
                 <geometry>
-                    <cylinder length="0.8068" radius="0.102"/>
+                    <cylinder length="0.754" radius="0.115"/>
                 </geometry>
                 <origin rpy="0 1.571 0"/>
@@ -12,35 +12,9 @@
                 </material>
             </visual>
-            <visual>
-                <geometry>
-                    <sphere radius="0.102"/>
-                </geometry>
-                <origin xyz="0.4034 0 0"/>
-                <material name="white"/>
-            </visual>
-            <visual>
-                <geometry>
-                    <sphere radius="0.102"/>
-                </geometry>
-                <origin xyz="-0.4034 0 0"/>
-                <material name="white"/>
-            </visual>
             <collision>
                 <geometry>
-                    <cylinder length="0.8068" radius="0.102"/>
+                    <cylinder length="0.754" radius="0.115"/>
                 </geometry>
                 <origin rpy="0 1.571 0"/>
-            </collision>
-            <collision>
-                <geometry>
-                    <sphere radius="0.102"/>
-                </geometry>
-                <origin xyz="0.4034 0 0"/>
-            </collision>
-            <collision>
-                <geometry>
-                    <sphere radius="0.102"/>
-                </geometry>
-                <origin xyz="-0.4034 0 0"/>
             </collision>
         </link>

File: ucf_sub/src/sub_definition/urdf/sub_thruster.urdf.xacro (robot description, xacro)
@@ -27,4 +27,22 @@
                 <origin xyz="0 0 -0.0522" rpy="1.571 0 0"/>
             </visual>
+            <collision>
+                <geometry>
+                    <cylinder length="0.131" radius="0.02"/>
+                </geometry>
+                <origin rpy="0 -1.571 0" xyz="0.0253 0 0"/>
+            </collision>
+            <collision>
+                <geometry>
+                    <cylinder length="0.0445" radius="0.0458"/>
+                </geometry>
+                <origin rpy="0 -1.571 0" xyz="0 0 0"/>
+            </collision>
+            <collision>
+                <geometry>
+                    <box size="0.0634 0.0128 0.0381"/>
+                </geometry>
+                <origin xyz="0 0 -0.0522" rpy="1.571 0 0"/>
+            </collision>
         </link>
         <joint name="${identifier}_thruster_joint" type="fixed">

File: ucf_sub/src/sub_definition/urdf/vision_cam.urdf.xacro (robot description, xacro)
@@ -16,4 +16,11 @@
             </visual>
         </link>
+	<sensor name="${identifier}_cam_sensor" update_rate="30">
+		<parent link="${identifier}_cam_sensor"/>
+		<origin xyz="0 0 0" rpy="0 0 0"/>
+		<camera>
+			<image width="1288" height="964" hfov="1.571" near="0.01" far="50.0"/>
+		</camera>
+	</sensor>
         <joint name="${identifier}_cam_joint" type="fixed">
 			<parent link="${parent}"/>

Commit message: Updated robot urdf with imu and no arms

File: ucf_sub/src/sub_definition/robots/ucf_robosub.urdf.xacro (robot description, xacro)
@@ -1,20 +1,26 @@
 <?xml version="1.0"?>
 <robot name="ucf_robosub" xmlns:xacro="http://www.ros.org/wiki/xacro">
-    <xacro:include filename="$(find ucf_sub_definition)/urdf/sub_body.urdf.xacro"/>
-    <xacro:include filename="$(find ucf_sub_definition)/urdf/sub_thruster.urdf.xacro"/>
-    <xacro:include filename="$(find ucf_sub_definition)/urdf/sub_arm.urdf.xacro"/>
-    <xacro:include filename="$(find ucf_sub_definition)/urdf/vision_cam.urdf.xacro"/>
-    <sub_body />
-    <sub_thruster identifier="vertical1" parent="base_link" xPos="0.11" yPos="-0.18" zPos="0.0" roll="1.571" pitch="1.571" yaw="0.0"/>
-    <sub_thruster identifier="vertical2" parent="base_link" xPos="-0.08" yPos="-0.18" zPos="0.0" roll="1.571" pitch="1.571" yaw="0.0"/>
-    <sub_thruster identifier="vertical3" parent="base_link" xPos="-0.08" yPos="0.18" zPos="0.0" roll="-1.571" pitch="1.571" yaw="0.0"/>
-    <sub_thruster identifier="vertical4" parent="base_link" xPos="0.11" yPos="0.18" zPos="0.0" roll="-1.571" pitch="1.571" yaw="0.0"/>
-    <sub_thruster identifier="horizontal1" parent="base_link" xPos="0.24" yPos="-0.19" zPos="0.0" roll="-1.571" pitch="0.0" yaw="3.927"/>
-    <sub_thruster identifier="horizontal2" parent="base_link" xPos="-0.21" yPos="-0.19" zPos="0.0" roll="1.571" pitch="0.0" yaw="-0.785"/>
-    <sub_thruster identifier="horizontal3" parent="base_link" xPos="-0.21" yPos="0.19" zPos="0.0" roll="-1.571" pitch="0.0" yaw="0.785"/>
-    <sub_thruster identifier="horizontal4" parent="base_link" xPos="0.24" yPos="0.19" zPos="0.0" roll="1.571" pitch="0.0" yaw="-3.927"/>
-    <sub_arm identifier="right" parent="base_link" xPos="0.275" yPos="0.099" zPos="-0.0623" roll="0.0" pitch="0.0" yaw="0.0"/>
-    <sub_arm identifier="left" parent="base_link" xPos="0.275" yPos="-0.0482" zPos="-0.0623" roll="0.0" pitch="0.0" yaw="0.0"/>
+    <xacro:include filename="$(find sub_definition)/urdf/sub_body.urdf.xacro"/>
+    <xacro:include filename="$(find sub_definition)/urdf/sub_thruster.urdf.xacro"/>
+    <xacro:include filename="$(find sub_definition)/urdf/sub_arm.urdf.xacro"/>
+    <xacro:include filename="$(find sub_definition)/urdf/vision_cam.urdf.xacro"/>
+    <link name="base_link">
+    </link>
+    <sub_thruster identifier="vertical1" parent="base_link" xPos="0.105" yPos="-0.18" zPos="0.0" roll="1.571" pitch="0.0" yaw="1.571"/>
+    <sub_thruster identifier="vertical2" parent="base_link" xPos="0.105" yPos="0.18" zPos="0.0" roll="1.571" pitch="3.141" yaw="1.571"/>
+    <sub_thruster identifier="vertical3" parent="base_link" xPos="-0.105" yPos="0.18" zPos="0.0" roll="1.571" pitch="3.141" yaw="1.571"/>
+    <sub_thruster identifier="vertical4" parent="base_link" xPos="-0.105" yPos="-0.18" zPos="0.0" roll="1.571" pitch="0.0" yaw="1.571"/>
+    <sub_thruster identifier="horizontal1" parent="base_link" xPos="0.22" yPos="-0.18" zPos="0.0" roll="1.571" pitch="0.7855" yaw="3.141"/>
+    <sub_thruster identifier="horizontal2" parent="base_link" xPos="0.22" yPos="0.18" zPos="0.0" roll="-1.571" pitch="0.7855" yaw="3.141"/>
+    <sub_thruster identifier="horizontal3" parent="base_link" xPos="-0.22" yPos="0.18" zPos="0.0" roll="-1.571" pitch="-0.7855" yaw="0.0"/>
+    <sub_thruster identifier="horizontal4" parent="base_link" xPos="-0.22" yPos="-0.18" zPos="0.0" roll="1.571" pitch="-0.7855" yaw="0.0"/>
     <sub_vision_cam identifier="left" parent="base_link" xPos="0.301" yPos="-0.051" zPos="0.0" roll="0.0" pitch="0.0" yaw="0.0"/>
     <sub_vision_cam identifier="right" parent="base_link" xPos="0.301" yPos="0.051" zPos="0.0" roll="0.0" pitch="0.0" yaw="0.0"/>
+    <link name="ahrs8_imu">
+    </link>
+    <joint name="imu_joint" type="fixed">
+        <parent link="base_link"/>
+		<child link="ahrs8_imu"/>
+		<origin xyz="0.0 0.066 0.0" rpy="0.0 0.0 0.0"/>
+    </joint>
 </robot>

File: ucf_sub/src/sub_definition/test.urdf (robot description, URDF)
Before this commit: robot ucf_robosub, 15 links, 14 joints
Links:
- removed link base_link
- removed link left_arm_base
- removed link left_arm_main
- removed link right_arm_base
- removed link right_arm_main
- added link imu
- link horizontal1_thruster: geometry collision box size=0.0634 0.0128 0.0381; collision cylinder length=0.0445 radius=0.0458
- link horizontal2_thruster: geometry collision box size=0.0634 0.0128 0.0381; collision cylinder length=0.0445 radius=0.0458
- link horizontal3_thruster: geometry collision box size=0.0634 0.0128 0.0381; collision cylinder length=0.0445 radius=0.0458
- link horizontal4_thruster: geometry collision box size=0.0634 0.0128 0.0381; collision cylinder length=0.0445 radius=0.0458
- link vertical1_thruster: geometry collision box size=0.0634 0.0128 0.0381; collision cylinder length=0.0445 radius=0.0458
- link vertical2_thruster: geometry collision box size=0.0634 0.0128 0.0381; collision cylinder length=0.0445 radius=0.0458
- link vertical3_thruster: geometry collision box size=0.0634 0.0128 0.0381; collision cylinder length=0.0445 radius=0.0458
- link vertical4_thruster: geometry collision box size=0.0634 0.0128 0.0381; collision cylinder length=0.0445 radius=0.0458
Joints:
- removed joint left_arm_base_joint
- removed joint left_arm_pivot_joint
- removed joint right_arm_base_joint
- removed joint right_arm_pivot_joint
- added joint imu_joint: type None, parent base_link, child imu, origin xyz=0.0 0.066 0.0 rpy=0.0 0.0 0.0
- joint horizontal1_thruster_joint: origin xyz=0.24 -0.19 0.0 rpy=-1.571 0.0 3.927 -> xyz=0.22 -0.18 0.0 rpy=1.571 0.7855 3.141
- joint horizontal2_thruster_joint: origin xyz=-0.21 -0.19 0.0 rpy=1.571 0.0 -0.785 -> xyz=0.22 0.18 0.0 rpy=-1.571 0.7855 3.141
- joint horizontal3_thruster_joint: origin xyz=-0.21 0.19 0.0 rpy=-1.571 0.0 0.785 -> xyz=-0.22 0.18 0.0 rpy=-1.571 -0.7855 0.0
- joint horizontal4_thruster_joint: origin xyz=0.24 0.19 0.0 rpy=1.571 0.0 -3.927 -> xyz=-0.22 -0.18 0.0 rpy=1.571 -0.7855 0.0
- joint left_cam_joint: origin xyz=0.273 -0.0508 0.0 rpy=0.0 0.0 0.0 -> xyz=0.301 -0.051 0.0 rpy=0.0 0.0 0.0
- joint right_cam_joint: origin xyz=0.273 0.0508 0.0 rpy=0.0 0.0 0.0 -> xyz=0.301 0.051 0.0 rpy=0.0 0.0 0.0
- joint vertical1_thruster_joint: origin xyz=0.11 -0.18 0.0 rpy=1.571 1.571 0.0 -> xyz=0.105 -0.18 0.0 rpy=1.571 0.0 1.571
- joint vertical2_thruster_joint: origin xyz=-0.08 -0.18 0.0 rpy=1.571 1.571 0.0 -> xyz=0.105 0.18 0.0 rpy=1.571 3.141 1.571
- joint vertical3_thruster_joint: origin xyz=-0.08 0.18 0.0 rpy=-1.571 1.571 0.0 -> xyz=-0.105 0.18 0.0 rpy=1.571 3.141 1.571
- joint vertical4_thruster_joint: origin xyz=0.11 0.18 0.0 rpy=-1.571 1.571 0.0 -> xyz=-0.105 -0.18 0.0 rpy=1.571 0.0 1.571

File: ucf_sub/src/sub_definition/urdf/sub_arm.urdf.xacro (robot description, xacro)
@@ -28,5 +28,5 @@
 		    <origin xyz="-0.0191 -0.0254 -0.076" rpy="0 0 0"/>
 		    <axis xyz="0 1 0"/>
-		    <limit effort="2.8" lower="-1.57" upper="0.2" velocity="20"/>
+		    <limit effort="2.8" lower="-0.2" upper="1.57" velocity="20"/>
 		</joint>
     </xacro:macro>

Commit message: Added depth sensor to URDF

File: ucf_sub/src/sub_definition/robots/ucf_robosub.urdf.xacro (robot description, xacro)
@@ -21,6 +21,13 @@
     <joint name="imu_joint" type="fixed">
         <parent link="base_link"/>
-		<child link="ahrs8_imu"/>
-		<origin xyz="0.0 0.066 0.0" rpy="0.0 0.0 0.0"/>
+	<child link="ahrs8_imu"/>
+	<origin xyz="0.0 0.066 0.0" rpy="0.0 0.0 0.0"/>
+    </joint>
+    <link name="depth">
+    </link>
+    <joint name="depth_joint" type="fixed">
+        <parent link="base_link"/>
+        <child link="depth"/>
+        <origin xyz="-0.3 -0.2 0.0" rpy="0.0 0.0 0.0"/>
     </joint>
 </robot>
