Commit message: So much bug smashing

File: ucf_sub_catkin_ros/src/sub_definition/robots/ucf_robosub.urdf.xacro (robot description, xacro)
@@ -22,5 +22,5 @@
         <parent link="base_link"/>
 	<child link="ahrs8_imu"/>
-	<origin xyz="0.0 0.066 0.0" rpy="0.0 0.0 0.0"/>
+	<origin xyz="0.0 0.066 0.0" rpy="3.141 0.0 3.141"/>
     </joint>
     <link name="depth">
